File: SL_MicroUSB-Breakout/SL_MicroUSB-Breakout.kicad_pcb (KiCad board)
At the start: 2 copper layers, 17 x 20 mm, 7 parts, among them J1 USB_B_Micro, J2 Conn_01x01, J3 Conn_01x01, J4 Conn_01x05_Male

Commit message: fix pin 1 marking
Parts:
- J4: moved to B.Cu
- moved J4 10.1 mm to (150.0, 111.6)
Connections:
- J4 pad 1: /GND -> /5V
- J4 pad 2: /ID -> /D-
- J4 pad 4: /D- -> /ID
- J4 pad 5: /5V -> /GND
Changed lines of the file:
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@@
-    )
-  )
-  (footprint "Connector_PinHeader_2.54mm:PinHeader_1x05_P2.54mm_Vertical" (layer "F.Cu")
-    (at 139.925 111.5 90)
-    (descr "Through hole straight pin header, 1x05, 2.54mm pitch, single row")
-    (tags "Through hole pin header THT 1x05 2.54mm single row")
-    (property "Sheetfile" "SL_MicroUSB-Breakout.kicad_sch")
-    (property "Sheetname" "")
-    (attr through_hole)
-    (fp_text reference "J4" (at 0 -2.33 90) (layer "F.SilkS") hide
-      (effects (font (size 1 1) (thickness 0.15)))
-    )
-    (fp_text value "Conn_01x05_Male" (at -3 5.075 180) (layer "F.Fab")
-      (effects (font (size 1 1) (thickness 0.15)))
-    )
-    (fp_text user "${REFERENCE}" (at 0 5.08) (layer "F.Fab")
-      (effects (font (size 1 1) (thickness 0.15)))
-    )
-    (fp_line (start -1.33 -1.33) (end 0 -1.33) (layer "F.SilkS") (width 0.12))
-    (fp_line (start -1.33 0) (end -1.33 -1.33) (layer "F.SilkS") (width 0.12))
-    (fp_line (start -1.33 1.27) (end 1.33 1.27) (layer "F.SilkS") (width 0.12))
-    (fp_line (start -1.33 1.27) (end -1.33 11.49) (layer "F.SilkS") (width 0.12))
-    (fp_line (start -1.33 11.49) (end 1.33 11.49) (layer "F.SilkS") (width 0.12))
-    (fp_line (start 1.33 1.27) (end 1.33 11.49) (layer "F.SilkS") (width 0.12))
-    (fp_line (start -1.8 -1.8) (end -1.8 11.95) (layer "F.CrtYd") (width 0.05))
-    (fp_line (start -1.8 11.95) (end 1.8 11.95) (layer "F.CrtYd") (width 0.05))
-    (fp_line (start 1.8 -1.8) (end -1.8 -1.8) (layer "F.CrtYd") (width 0.05))
-    (fp_line (start 1.8 11.95) (end 1.8 -1.8) (layer "F.CrtYd") (width 0.05))
-    (fp_line (start -1.27 11.43) (end -1.27 -0.635) (layer "F.Fab") (width 0.1))
-    (fp_line (start 1.27 -1.27) (end 1.27 11.43) (layer "F.Fab") (width 0.1))
-    (fp_line (start -0.635 -1.27) (end 1.27 -1.27) (layer "F.Fab") (width 0.1))
-    (fp_line (start -1.27 -0.635) (end -0.635 -1.27) (layer "F.Fab") (width 0.1))
-    (fp_line (start 1.27 11.43) (end -1.27 11.43) (layer "F.Fab") (width 0.1))
-    (pad "1" thru_hole rect (at 0 0 90) (size 1.7 1.7) (drill 1) (layers *.Cu *.Mask)
-      (net 5 "/GND") (pinfunction "Pin_1") (pintype "passive"))
-    (pad "2" thru_hole oval (at 0 2.54 90) (size 1.7 1.7) (drill 1) (layers *.Cu *.Mask)
-      (net 4 "/ID") (pinfunction "Pin_2") (pintype "passive"))
-    (pad "3" thru_hole oval (at 0 5.08 90) (size 1.7 1.7) (drill 1) (layers *.Cu *.Mask)
-      (net 2 "/D+") (pinfunction "Pin_3") (pintype "passive"))
-    (pad "4" thru_hole oval (at 0 7.62 90) (size 1.7 1.7) (drill 1) (layers *.Cu *.Mask)
-      (net 3 "/D-") (pinfunction "Pin_4") (pintype "passive"))
-    (pad "5" thru_hole oval (at 0 10.16 90) (size 1.7 1.7) (drill 1) (layers *.Cu *.Mask)
-      (net 1 "/5V") (pinfunction "Pin_5") (pintype "passive"))
-    (model "${KICAD6_3DMODEL_DIR}/Connector_PinHeader_2.54mm.3dshapes/PinHeader_1x05_P2.54mm_Vertical.wrl"
-      (offset (xyz 0 0 0))
-      (scale (xyz 1 1 1))
-      (rotate (xyz 0 0 0))
     )
   )
@@
       (offset (xyz 0 0 0))
       (scale (xyz 1 1 1))
+      (rotate (xyz 0 0 0))
+    )
+  )
+  (footprint "Connector_PinHeader_2.54mm:PinHeader_1x05_P2.54mm_Vertical" (layer "B.Cu")
+    (at 150 111.6 90)
+    (descr "Through hole straight pin header, 1x05, 2.54mm pitch, single row")
+    (tags "Through hole pin header THT 1x05 2.54mm single row")
+    (property "Sheetfile" "SL_MicroUSB-Breakout.kicad_sch")
+    (property "Sheetname" "")
+    (attr through_hole)
+    (fp_text reference "J4" (at 0 2.33 90) (layer "B.SilkS") hide
+      (effects (font (size 1 1) (thickness 0.15)) (justify mirror))
+    )
+    (fp_text value "Conn_01x05_Male" (at -3 -5.075) (layer "B.Fab")
+      (effects (font (size 1 1) (thickness 0.15)) (justify mirror))
+    )
+    (fp_text user "${REFERENCE}" (at 0 -5.08) (layer "B.Fab")
+      (effects (font (size 1 1) (thickness 0.15)) (justify mirror))
+    )
+    (fp_line (start -1.33 1.33) (end 0 1.33) (layer "B.SilkS") (width 0.12))
+    (fp_line (start -1.33 0) (end -1.33 1.33) (layer "B.SilkS") (width 0.12))
+    (fp_line (start -1.33 -1.27) (end 1.33 -1.27) (layer "B.SilkS") (width 0.12))
+    (fp_line (start -1.33 -1.27) (end -1.33 -11.49) (layer "B.SilkS") (width 0.12))
+    (fp_line (start -1.33 -11.49) (end 1.33 -11.49) (layer "B.SilkS") (width 0.12))
+    (fp_line (start 1.33 -1.27) (end 1.33 -11.49) (layer "B.SilkS") (width 0.12))
+    (fp_line (start -1.8 1.8) (end -1.8 -11.95) (layer "B.CrtYd") (width 0.05))
+    (fp_line (start -1.8 -11.95) (end 1.8 -11.95) (layer "B.CrtYd") (width 0.05))
+    (fp_line (start 1.8 1.8) (end -1.8 1.8) (layer "B.CrtYd") (width 0.05))
+    (fp_line (start 1.8 -11.95) (end 1.8 1.8) (layer "B.CrtYd") (width 0.05))
+    (fp_line (start -1.27 -11.43) (end -1.27 0.635) (layer "B.Fab") (width 0.1))
+    (fp_line (start 1.27 1.27) (end 1.27 -11.43) (layer "B.Fab") (width 0.1))
+    (fp_line (start -0.635 1.27) (end 1.27 1.27) (layer "B.Fab") (width 0.1))
+    (fp_line (start -1.27 0.635) (end -0.635 1.27) (layer "B.Fab") (width 0.1))
+    (fp_line (start 1.27 -11.43) (end -1.27 -11.43) (layer "B.Fab") (width 0.1))
+    (pad "1" thru_hole rect (at 0 0 90) (size 1.7 1.7) (drill 1) (layers *.Cu *.Mask)
+      (net 1 "/5V") (pinfunction "Pin_1") (pintype "passive"))
+    (pad "2" thru_hole oval (at 0 -2.54 90) (size 1.7 1.7) (drill 1) (layers *.Cu *.Mask)
+      (net 3 "/D-") (pinfunction "Pin_2") (pintype "passive"))
+    (pad "3" thru_hole oval (at 0 -5.08 90) (size 1.7 1.7) (drill 1) (layers *.Cu *.Mask)
+      (net 2 "/D+") (pinfunction "Pin_3") (pintype "passive"))
+    (pad "4" thru_hole oval (at 0 -7.62 90) (size 1.7 1.7) (drill 1) (layers *.Cu *.Mask)
+      (net 4 "/ID") (pinfunction "Pin_4") (pintype "passive"))
+    (pad "5" thru_hole oval (at 0 -10.16 90) (size 1.7 1.7) (drill 1) (layers *.Cu *.Mask)
+      (net 5 "/GND") (pinfunction "Pin_5") (pintype "passive"))
+    (model "${KICAD6_3DMODEL_DIR}/Connector_PinHeader_2.54mm.3dshapes/PinHeader_1x05_P2.54mm_Vertical.wrl"
+      (offset (xyz 0 0 0))
+      (scale (xyz 1 1 1))
