File: SL_MicroUSB-Breakout/SL_MicroUSB-Breakout.kicad_sch (KiCad schematic)
At the start: 6 parts, among them J1 USB_B_Micro, J2 Conn_01x01, J3 Conn_01x01, J4 Conn_01x05_Male

Commit message: fix pin 1 marking
Parts:
- J4: value Conn_01x05_Male -> (none)
Connections:
- net 5V: now also J4.1 (Pin_1); no longer J4.5 (Pin_5)
- net D-: now also J4.2 (Pin_2); no longer J4.4 (Pin_4)
- net GND: now also J4.5 (Pin_5); no longer J4.1 (Pin_1)
- net ID: now also J4.4 (Pin_4); no longer J4.2 (Pin_2)
Other:
- moved on the sheet: J4
Changed lines of the file:
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@@
     (effects (font (size 1.27 1.27)) (justify left bottom))
   )
-  (symbol (lib_id "Connector:Conn_01x05_Male") (at 140.97 100.33 180) (unit 1)
+  (symbol (lib_id "Connector:Conn_01x05_Male") (at 130.81 100.33 0) (unit 1)
     (in_bom yes) (on_board yes)
-    (property "Reference" "J4" (id 0) (at 142.24 99.0599 0)
+    (property "Reference" "J4" (id 0) (at 139.7 101.6 0)
       (effects (font (size 1.27 1.27)) (justify right))
     )
-    (property "Value" "Conn_01x05_Male" (id 1) (at 142.24 101.5999 0)
+    (property "Value" "" (id 1) (at 154.94 99.06 0)
       (effects (font (size 1.27 1.27)) (justify right))
     )
-    (property "Footprint" "Connector_PinHeader_2.54mm:PinHeader_1x05_P2.54mm_Vertical" (id 2) (at 140.97 100.33 0)
+    (property "Footprint" "Connector_PinHeader_2.54mm:PinHeader_1x05_P2.54mm_Vertical" (id 2) (at 130.81 100.33 0)
       (effects (font (size 1.27 1.27)) hide)
     )
-    (property "Datasheet" "~" (id 3) (at 140.97 100.33 0)
+    (property "Datasheet" "~" (id 3) (at 130.81 100.33 0)
       (effects (font (size 1.27 1.27)) hide)
     )

Commit message: added some notes
Parts:
- J4: value (none) -> Conn_01x05_Male
Other:
- company: (none) -> Sternenlabor e.V.
- title: (none) -> SL MicroUSB Breakout
